File: KiCad/Pwr.kicad_sch (KiCad schematic)
At the start: 7 parts, among them J2 USB_C_Receptacle_USB2.0_16P, SW10 SW_Slide_DPDT

Commit message: added hierachical sheets to controllers
Parts:
- removed J2: USB_C_Receptacle_USB2.0_16P, symbol CM5_HighSpeedBreakout:USB_C_Receptacle_USB2.0_16P
Changed lines of the file:
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@@
-	)
-	(symbol
-		(lib_id "CM5_HighSpeedBreakout:USB_C_Receptacle_USB2.0_16P")
-		(at 45.72 44.45 0)
-		(unit 1)
-		(exclude_from_sim no)
-		(in_bom yes)
-		(on_board yes)
-		(dnp no)
-		(fields_autoplaced yes)
-		(property "Reference" "J2"
-			(at 45.72 21.59 0)
-			(effects
-				(font
-					(size 1.27 1.27)
-				)
-			)
-		)
-		(property "Value" "USB_C_Receptacle_USB2.0_16P"
-			(at 45.72 24.13 0)
-			(effects
-				(font
-					(size 1.27 1.27)
-				)
-			)
-		)
-		(property "Footprint" ""
-			(at 49.53 44.45 0)
-			(effects
-				(font
-					(size 1.27 1.27)
-				)
-				(hide yes)
-			)
-		)
-		(property "Datasheet" "https://www.usb.org/sites/default/files/documents/usb_type-c.zip"
-			(at 49.53 44.45 0)
-			(effects
-				(font
-					(size 1.27 1.27)
-				)
-				(hide yes)
-			)
-		)
-		(property "Description" "USB 2.0-only 16P Type-C Receptacle connector"
-			(at 45.72 44.45 0)
-			(effects
-				(font
-					(size 1.27 1.27)
-				)
-				(hide yes)
-			)
-		)
-		(pin "A8"
-		)
-		(pin "B12"
-		)
-		(pin "B1"
-		)
-		(pin "B8"
-		)
-		(pin "B9"
-		)
-		(pin "A5"
-		)
-		(pin "A1"
-		)
-		(pin "S1"
-		)
-		(pin "A4"
-		)
-		(pin "A9"
-		)
-		(pin "B6"
-		)
-		(pin "B4"
-		)
-		(pin "A7"
-		)
-		(pin "B7"
-		)
-		(pin "A6"
-		)
-		(pin "B5"
-		)
-		(pin "A12"
-		)
-		(instances
-			(project "sb_handheld"
-				(path "/e2b47f54-afd4-414f-8c8f-251eedeb980e/a13c2f15-7cd7-4af9-b5b9-3924f59a5254"
-					(reference "J2")
-					(unit 1)
-				)
-			)
-		)
 	)
 	(symbol
