File: KiCad/sbc.kicad_sch (KiCad schematic)
At the start: 2 parts, among them SW5 SW_Push

Commit message: added hierachical sheets to controllers
Parts:
- removed SW5: SW_Push, symbol CM5_HighSpeedBreakout:SW_Push
Connections:
- net +3V3: now reaches Module1.84 (+3.3v_(Output))
- net +3V3: now also Module1.86 (+3.3v_(Output))
Other:
- note removed: "Home btn"
Changed lines of the file:
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@@
 	(generator_version "9.0")
 	(paper "A4")
-	(text "Home btn"
-		(exclude_from_sim no)
-		(at 128.778 175.006 0)
-		(effects
-			(font
-				(size 1.27 1.27)
-			)
-		)
-	)
 	(junction
 		(at 102.87 134.62)
@@
 	)
 	(junction
+		(at 36.83 142.24)
+		(diameter 0)
+		(color 0 0 0 0)
+	)
+	(junction
 		(at 102.87 137.16)
 		(diameter 0)
@@
 	(wire
 		(pts
+			(xy 36.83 144.78) (xy 36.83 142.24)
+		)
+		(stroke
+			(width 0)
+			(type default)
+		)
+	)
+	(wire
+		(pts
 			(xy 102.87 139.7) (xy 102.87 142.24)
 		)
@@
 	(wire
 		(pts
+			(xy 41.91 144.78) (xy 36.83 144.78)
+		)
+		(stroke
+			(width 0)
+			(type default)
+		)
+	)
+	(wire
+		(pts
 			(xy 102.87 137.16) (xy 102.87 139.7)
 		)
@@
 		(pts
 			(xy 118.11 134.62) (xy 118.11 133.35)
+		)
+		(stroke
+			(width 0)
+			(type default)
+		)
+	)
+	(wire
+		(pts
+			(xy 36.83 142.24) (xy 41.91 142.24)
 		)
 		(stroke
@@
 	)
 	(symbol
+		(lib_id "power:+3V3")
+		(at 36.83 142.24 0)
+		(unit 1)
+		(exclude_from_sim no)
+		(in_bom yes)
+		(on_board yes)
+		(dnp no)
+		(fields_autoplaced yes)
+		(property "Reference" "#PWR026"
+			(at 36.83 146.05 0)
+			(effects
+				(font
+					(size 1.27 1.27)
+				)
+				(hide yes)
+			)
+		)
+		(property "Value" "+3V3"
+			(at 36.83 137.16 0)
+			(effects
+				(font
+					(size 1.27 1.27)
+				)
+			)
+		)
+		(property "Footprint" ""
+			(at 36.83 142.24 0)
+			(effects
+				(font
+					(size 1.27 1.27)
+				)
+				(hide yes)
+			)
+		)
+		(property "Datasheet" ""
+			(at 36.83 142.24 0)
+			(effects
+				(font
+					(size 1.27 1.27)
+				)
+				(hide yes)
+			)
+		)
+		(property "Description" "Power symbol creates a global label with name \"+3V3\""
+			(at 36.83 142.24 0)
+			(effects
+				(font
+					(size 1.27 1.27)
+				)
+				(hide yes)
+			)
+		)
+		(pin "1"
+		)
+		(instances
+			(project ""
+				(path "/e2b47f54-afd4-414f-8c8f-251eedeb980e/54ad1413-ad8b-422f-86f7-54b541faf2f8"
+					(reference "#PWR026")
+					(unit 1)
+				)
+			)
+		)
+	)
+	(symbol
 		(lib_id "power:GND")
 		(at 113.03 91.44 0)
@@
 					(unit 1)
 				)
-			)
-		)
-	)
-	(symbol
-		(lib_id "CM5_HighSpeedBreakout:SW_Push")
-		(at 143.51 182.88 0)
-		(unit 1)
-		(exclude_from_sim no)
-		(in_bom yes)
-		(on_board yes)
-		(dnp no)
-		(fields_autoplaced yes)
-		(property "Reference" "SW5"
-			(at 143.51 175.26 0)
-			(effects
-				(font
-					(size 1.27 1.27)
-				)
-			)
-		)
-		(property "Value" "SW_Push"
-			(at 143.51 177.8 0)
-			(effects
-				(font
-					(size 1.27 1.27)
-				)
-			)
-		)
-		(property "Footprint" ""
-			(at 143.51 177.8 0)
-			(effects
-				(font
-					(size 1.27 1.27)
-				)
-				(hide yes)
-			)
-		)
-		(property "Datasheet" "~"
-			(at 143.51 177.8 0)
-			(effects
-				(font
-					(size 1.27 1.27)
-				)
-				(hide yes)
-			)
-		)
-		(property "Description" "Push button switch, generic, two pins"
-			(at 143.51 182.88 0)
-			(effects
-				(font
-					(size 1.27 1.27)
-				)
-				(hide yes)
-			)
-		)
-		(pin "1"
-		)
-		(pin "2"
-		)
-		(instances
-			(project "sb_handheld"
-				(path "/e2b47f54-afd4-414f-8c8f-251eedeb980e/54ad1413-ad8b-422f-86f7-54b541faf2f8"
-					(reference "SW5")
-					(unit 1)
-				)

Commit message: redid button pull up. Added initial joystick and display symbols
Connections:
- no-connect marks 0 -> 11
Changed lines of the file:
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@@
 		(color 0 0 0 0)
+	)
+	(no_connect
+		(at 41.91 127)
+	)
+	(no_connect
+		(at 102.87 124.46)
+	)
+	(no_connect
+		(at 41.91 124.46)
+	)
+	(no_connect
+		(at 102.87 129.54)
+	)
+	(no_connect
+		(at 102.87 121.92)
+	)
+	(no_connect
+		(at 102.87 114.3)
+	)
+	(no_connect
+		(at 102.87 132.08)
+	)
+	(no_connect
+		(at 41.91 121.92)
+	)
+	(no_connect
+		(at 41.91 116.84)
+	)
+	(no_connect
+		(at 41.91 114.3)
+	)
+	(no_connect
+		(at 102.87 116.84)
 	)
 	(wire
